File: forty_mate.kicad_pcb (KiCad board)
At the start: 2 copper layers, 247.7 x 76.2 mm, 99 parts, among them SW1 SW_Push, SW10 SW_Push, SW11 SW_Push, SW12 SW_Push, SW13 SW_Push, SW14 SW_Push, SW15 SW_Push, SW16 SW_Push, SW17 SW_Push, SW18 SW_Push, SW19 SW_Push, SW2 SW_Push, SW20 SW_Push, SW21 SW_Push, SW22 SW_Push, SW23 SW_Push, SW24 SW_Push, SW25 SW_Push, SW26 SW_Push, SW27 SW_Push, SW28 SW_Push, SW29 SW_Push, SW3 SW_Push, SW30 SW_Push, SW31 SW_Push, SW32 SW_Push, SW33 SW_Push, SW34 SW_Push, SW35 SW_Push, SW36 SW_Push, SW37 SW_Push, SW38 SW_Push, SW39 SW_Push, SW4 SW_Push, SW40 SW_Push, SW41 SW_Push, SW42 SW_Push, SW43 SW_Push, SW44 SW_SPDT, SW45 SW_Push, SW5 SW_Push, SW6 SW_Push, SW7 SW_Push, SW8 SW_Push, SW9 SW_Push, U1 Micon_BLEMicroPro

Commit message: modify copper pattern
Routing:
- net row2: track 307.9 -> 309.5 mm
- net col0: track 266.2 -> 267.3 mm
- net row1: track 299.7 -> 298.6 mm
- net col1: track 270.0 -> 270.9 mm
- net col10: track 158.4 -> 159.3 mm
- net col6: track 326.8 -> 327.5 mm
- net col7: track 157.3 -> 158.0 mm
- net col5: track 339.6 -> 340.2 mm
- net col2: track 254.2 -> 254.7 mm
